File: fluke_752A_pcb.kicad_pcb (KiCad board)
At the start: 2 copper layers, 76 parts, among them J1 F, J10 J, J11 K, J12 L, J13 M, J14 N, J15 O, J16 P, J17 Q, J18 R, J19 S, J2 H, J20 T1, J21 T2, J22 T4, J23 T3, J24 U, J25 V4, J26 V7, J27 V1, J28 V6, J29 V2, J3 A, J30 V3, J31 V5, J32 V8, J33 V9, J4 B, J5 C, J6 D, J7 E, J8 G, J9 I

Commit message: PCB Version 2
Parts:
- removed the J25 at (198.1, 151.1)
- removed the J26 at (228.6, 137.2)
- removed the J27 at (165.1, 137.2)
- removed J28: V6, fluke_752A_pcb_specific_components:PTFE pins
- removed J29: V2, fluke_752A_pcb_specific_components:PTFE pins
- removed J30: V3, fluke_752A_pcb_specific_components:PTFE pins
- removed J31: V5, fluke_752A_pcb_specific_components:PTFE pins
- removed J32: V8, fluke_752A_pcb_specific_components:PTFE pins
- removed J33: V9, fluke_752A_pcb_specific_components:PTFE pins
- JP1: renamed from JP7; value jpr -> (none)
- JP10: renamed from JP5; value jpr -> (none)
- JP11: value jpr -> (none)
- JP12: renamed from JP13; value jpr -> (none)
- JP13: renamed from JP12; value jpr -> (none)
- JP14: renamed from JP15; value jpr -> (none)
- JP15: renamed from JP16; value jpr -> (none)
- JP16: renamed from JP14; value jpr -> (none)
- JP2: renamed from JP6; value jpr -> (none)
- JP3: renamed from JP8; value jpr -> (none)
- JP4: renamed from JP10; value jpr -> (none)
- JP5: renamed from JP9; value jpr -> (none)
- JP6: renamed from JP3; value jpr -> (none)
- JP7: renamed from JP1; value jpr -> (none)
- JP8: renamed from JP2; value jpr -> (none)
- JP9: renamed from JP4; value jpr -> (none)
- R4: renamed from R24; value R -> 15
- R401: renamed from R2; value R -> 60
- R402: renamed from R3; value R -> 60
- R403: renamed from R4; value R -> 90
- R404: renamed from R6; value R -> 30
- R405: renamed from R5; value R -> 300
- R42: renamed from R12; value R -> 48
- R43: renamed from R8; value R -> 2k
- R44: renamed from R7; value R -> 1k
- R45: renamed from R9; value R -> 500
- R46: renamed from R11; value R -> 250
- R47: renamed from R10; value R -> 125
- R48: renamed from R14; value R -> 60
- R5: renamed from R21; value R -> 15
- R50: renamed from R13; value R -> 200
- R502: renamed from R19; value R -> 10
- R503: renamed from R18; value R -> 10
- R504: renamed from R27; value R -> 15
- R506: renamed from R26; value R -> 250
- R507: renamed from R25; value R -> 1k
- R6: renamed from R22; value R -> 15
- renumbered J20 to ?, J22 to ?, J3 to J1, J24 to J14, J21 to J15, J23 to J16, J19 to J17, J17 to J19, J4 to J2, J16 to J20, J15 to J21, J14 to J22, J13 to J23, J12 to J24, J11 to J25, J10 to J26, J9 to J27, J5 to J3, J6 to J4, J7 to J5, J1 to J6, J8 to J7, J2 to J8, R20 to R25, R23 to R35, R1 to R41, R16 to R501, R17 to R508, R15 to R509
Routing:
- net GND: vias 8 -> 0
Other:
- board outline added: 255.1 x 141.1 mm
- board text added: "10"
- board text added: "11"
- board text added: "12"
- board text added: "13"
- board text added: "9"
- board text added: "E1"
- board text added: "E10"
- board text added: "E11"
- board text added: "E12"
- board text added: "E13"
- board text added: "E14"
- board text added: "E15"
- board text added: "E16"
- board text added: "E17"
- board text added: "E18"
- board text added: "E19"
- board text added: "E2"
- board text added: "E20"
- board text added: "E21"
- board text added: "E22"
- board text added: "E23"
- board text added: "E24"
- board text added: "E25"
- board text added: "E26"
- board text added: "E27"
- board text added: "E28"
- board text added: "E29"
- board text added: "E3"
- board text added: "E30"
- board text added: "E4"
- board text added: "E5"
- board text added: "E6"
- board text added: "E7"
- board text added: "E8"
- board text added: "E9"
- board text added: "R25"
- board text added: "R35"
- board text added: "R4"
- board text added: "R401"
- board text added: "R402"
- board text added: "R403"
- board text added: "R404"
- board text added: "R405"
- board text added: "R41"
- board text added: "R42"
- board text added: "R43"
- board text added: "R44"
- board text added: "R45"
- board text added: "R46"
- board text added: "R47"
- board text added: "R48"
- board text added: "R5"
- board text added: "R50"
- board text added: "R501"
- board text added: "R502"
- board text added: "R503"
- board text added: "R504"
- board text added: "R506"
- board text added: "R507"
- board text added: "R508"
- board text added: "R509"
- board text added: "R6"
- board text added: "R601"
- board text added: "R602"
- board text added: "R603"
- board text added: "R604"
- board text added: "R605"
- board text added: "R606"
- board text added: "R607"
- board text added: "R608"
